File: board/balancing.kicad_sch (KiCad schematic)
At the start: 7 parts, among them U4 ETA3000S2G

Commit message: incorporate review feedback
Parts:
- L2: footprint Inductor_SMD:L_Bourns_SRP7028A_7.3x6.6mm -> Inductor_SMD:L_Bourns-SRN4018
Changed lines of the file:
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@@
       (effects (font (size 1.27 1.27)))
     )
-    (property "Footprint" "Inductor_SMD:L_Bourns_SRP7028A_7.3x6.6mm" (at 151.13 81.28 0)
+    (property "Footprint" "Inductor_SMD:L_Bourns-SRN4018" (at 151.13 81.28 0)
       (effects (font (size 1.27 1.27)) hide)
     )
